Commit message: Driven the bot

File: description/robot_core.xacro (robot description, xacro)
@@ -41,4 +41,7 @@
         </xacro:inertial_box>
     </link>
+    <gazebo reference="chasis">
+    	<material>Gazebo/White</material>
+    </gazebo>
     <!-- LEFT WHEEl-->
     <joint name="left_wheel_joint" type="continuous">
@@ -64,4 +67,7 @@
         </xacro:inertial_cylinder>
     </link>
+    <gazebo reference="left_wheel">
+    	<material>Gazebo/Blue</material>
+    </gazebo>
      <!-- right WHEEl-->
      <joint name="right_wheel_joint" type="continuous">
@@ -87,4 +93,7 @@
         </xacro:inertial_cylinder>
     </link>
+    <gazebo reference="right_wheel">
+    	<material>Gazebo/Blue</material>
+    </gazebo>
     <!-- Caster-->
     <joint name="caster_wheel_joint" type="fixed">
@@ -109,3 +118,8 @@
         </xacro:inertial_sphere>
     </link>
+    <gazebo reference="caster_wheel">
+    	<material>Gazebo/Black</material>
+        <mu1 value="0.001"/>
+        <mu2 value="0.002"/>
+    </gazebo>
 </robot>
